Commit message: 添加rgbd传感器

File: suv_description/urdf/gazebo/link_color.xacro (robot description, xacro)
@@ -27,3 +27,6 @@
         <material>Gazebo/White</material>
     </gazebo>
+    <gazebo reference="ZED_link">
+        <material>Gazebo/Grey</material>
+    </gazebo>
 </robot>

File: suv_description/urdf/suv.xacro (robot description, xacro)
@@ -4,5 +4,6 @@
     <xacro:include filename="$(find suv_description)/urdf/gazebo/link_color.xacro" />
     <xacro:include filename="$(find suv_description)/urdf/gazebo/imu.xacro" />
-<!-- *************************************************参数定义******************************************************* -->
+    <xacro:include filename="$(find suv_description)/urdf/gazebo/rgbd.xacro" />
+<!-- *****************************************参数定义************************************************ -->
     <!-- 质心到前轴距离 -->
     <xacro:property name="massCenter_to_Faxis" value="0.28" />
@@ -27,5 +28,5 @@
     <!-- 车体重量 -->
     <xacro:property name="car_weight" value="30.24" />
-<!-- *************************************************颜色定义******************************************************* -->
+<!-- ******************************************颜色定义************************************************ -->
     <xacro:property name="Green">
         <material name="Green">
@@ -53,5 +54,5 @@
         </material>
     </xacro:property>
-<!-- ************************************************base_link***************************************************** -->
+<!-- *****************************************base_link********************************************** -->
     <link name="base_footprint"></link>
     <joint name="base_link_to_footprint" type="fixed">
@@ -81,5 +82,5 @@
         </inertial>
     </link>
-<!-- **************************************************四个轮子***************************************************** -->
+<!-- *******************************************四个轮子********************************************** -->
     <!-- 后轮宏定义，y代表轮子所处象限,1为左，-1为右 -->
     <xacro:macro name="RearWheel" params="wheel_name y">
@@ -177,5 +178,5 @@
     <xacro:FrontWheel wheel_name="left_front" y="1" />
     <xacro:FrontWheel wheel_name="right_front" y="-1" />
-<!-- **************************************************传感器link************************************************** -->
+<!-- *******************************************传感器link******************************************* -->
     <!-- imu -->
     <joint name="imu_joint" type="fixed">
@@ -211,5 +212,5 @@
         <child link="ZED_link" />
         <axis xyz="0 0 0" />
-      </joint>
+    </joint>
     <link name="ZED_link">
         <inertial>
@@ -233,4 +234,4 @@
             </geometry>
         </collision>
-      </link>
+    </link>
 </robot>
